File: power-wing.brd (EAGLE design)
At the start: 50.8 x 22.9 mm, 25 parts, among them Q1 MOSFET-PGDS_TO220V, T1 2N2222, T2 2N2222, T3 2N2222, U1 TLV2462IP, U2 LD1117

Commit message: off switch to GPIO11 instead of 12 since that is used for sleep
Connections:
- removed net N$19: MS1.23
- new net GPIO11: MS1.23, R3.2
- net GPIO12: no longer R3.2
Routing:
- net GPIO11: track 0.00 -> 7.87 mm
- net GPIO12: track 5.18 -> 0.00 mm
Other:
- board text added: "V2"
Changed lines of the file:
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@@
 <text x="7.366" y="18.796" size="0.8128" layer="21">GND</text>
 <text x="14.224" y="20.32" size="0.8128" layer="21" rot="R90">VIN</text>
+<text x="46.736" y="5.842" size="0.17018125" layer="16" font="vector" rot="MR0">V2</text>
+<text x="46.736" y="5.588" size="1.27" layer="25" font="vector">V2</text>
 </plain>
 <attributes>
@@
 <signal name="GPIO12">
 <contactref element="MS1" pad="24"/>
-<contactref element="R3" pad="2"/>
-<wire x1="22.86" y1="18.288" x2="24.384" y2="19.812" width="0.4064" layer="1"/>
-<wire x1="24.384" y1="19.812" x2="24.892" y2="19.812" width="0.4064" layer="1"/>
-<wire x1="24.892" y1="19.812" x2="26.67" y2="21.59" width="0.4064" layer="1"/>
-</signal>
-<signal name="N$19">
-<contactref element="MS1" pad="23"/>
 </signal>
 <signal name="N$20">
@@
 <wire x1="30.988" y1="17.526" x2="30.226" y2="18.288" width="0.4064" layer="1"/>
 </signal>
+<signal name="GPIO11">
+<contactref element="R3" pad="2"/>
+<contactref element="MS1" pad="23"/>
+<wire x1="22.86" y1="18.288" x2="24.384" y2="19.812" width="0.4064" layer="16"/>
+<wire x1="24.384" y1="19.812" x2="27.686" y2="19.812" width="0.4064" layer="16"/>
+<wire x1="27.686" y1="19.812" x2="29.21" y2="21.336" width="0.4064" layer="16"/>
+<wire x1="29.21" y1="21.336" x2="29.21" y2="21.59" width="0.4064" layer="16"/>
+</signal>
 </signals>

Commit message: lets use some smaller parts
Parts:
- removed Q1: MOSFET-PGDS_TO220V, adafruit:TO220V
- removed U2: LD1117, dm_parts:TO220S
- added U$2: L4931, dm_parts:TO92-BCE
- added U$3: VP2206N3-G, dm_parts:TO92-BCE
Connections:
- net 3V: now also U$2.E; no longer U2.2
- net GND: now also U$2.C; no longer U2.1
- net N$16: now also U$3.C; no longer Q1.1
- net VIN: now also U$3.B; no longer Q1.3
- net VOUT: now also U$2.B, U$3.E; no longer Q1.2, U2.3
Routing:
- net N$16: track 19.6 -> 16.2 mm
- net VIN: track 16.8 -> 19.6 mm
Changed lines of the file:
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@@
 <attribute name="VALUE" x="38.862" y="11.811" size="1.27" layer="27" ratio="10"/>
-</element>
-<element name="Q1" library="adafruit" package="TO220V" value="MOSFET-PGDS_TO220V" x="4.318" y="9.144" smashed="yes">
-<attribute name="NAME" x="-0.762" y="3.0988" size="1.27" layer="25" ratio="10"/>
-<attribute name="VALUE" x="-0.762" y="1.524" size="1.27" layer="27" ratio="10"/>
 </element>
 <element name="C2" library="adafruit" package="E1,8-4" value="10u" x="19.558" y="14.732" smashed="yes" rot="R270">
@@
 <attribute name="VALUE" x="13.208" y="24.257" size="1.27" layer="27" rot="R180"/>
 </element>
-<element name="U2" library="dm_parts" package="TO220S" value="LD1117" x="15.24" y="2.794" smashed="yes" rot="R180">
-<attribute name="NAME" x="11.2522" y="5.334" size="1.27" layer="25" ratio="10" rot="R90"/>
-<attribute name="VALUE" x="20.32" y="10.414" size="1.27" layer="27" ratio="10" rot="R180"/>
-</element>
 <element name="C4" library="adafruit" package="C025-024X044" value=".1u" x="23.114" y="4.826" smashed="yes" rot="R270">
 <attribute name="NAME" x="24.511" y="6.604" size="1.27" layer="25" ratio="10" rot="R270"/>
@@
 <attribute name="VALUE" x="39.37" y="15.621" size="1.27" layer="27"/>
 </element>
+<element name="U$2" library="dm_parts" package="TO92-BCE" value="L4931" x="15.748" y="5.08"/>
+<element name="U$3" library="dm_parts" package="TO92-BCE" value="VP2206N3-G" x="7.112" y="6.096" rot="R180"/>
 </elements>
 <signals>
@@
 </polygon>
 <contactref element="JP2" pad="2"/>
-<contactref element="U2" pad="1"/>
 <contactref element="C4" pad="2"/>
 <contactref element="C5" pad="-"/>
 <contactref element="R9" pad="1"/>
+<contactref element="U$2" pad="C"/>
 </signal>
 <signal name="AREF">
@@
 <signal name="3V">
 <contactref element="MS1" pad="2"/>
-<contactref element="U2" pad="2"/>
 <contactref element="C5" pad="+"/>
 <wire x1="8.89" y1="1.27" x2="8.89" y2="2.794" width="0.4064" layer="1"/>
 <wire x1="8.89" y1="2.794" x2="9.144" y2="3.048" width="0.4064" layer="1"/>
-<wire x1="9.144" y1="3.048" x2="14.224" y2="3.048" width="0.4064" layer="1"/>
-<wire x1="14.224" y1="3.048" x2="14.478" y2="3.048" width="0.4064" layer="1"/>
-<wire x1="14.478" y1="3.048" x2="15.24" y2="3.81" width="0.4064" layer="1"/>
-<wire x1="15.24" y1="3.81" x2="15.24" y2="5.334" width="0.4064" layer="1"/>
+<wire x1="18.542" y1="3.048" x2="18.796" y2="3.048" width="0.4064" layer="1"/>
 <wire x1="27.559" y1="4.572" x2="24.384" y2="4.572" width="0.4064" layer="1"/>
 <wire x1="24.384" y1="4.572" x2="24.13" y2="4.826" width="0.4064" layer="1"/>
 <wire x1="24.13" y1="4.826" x2="20.574" y2="4.826" width="0.4064" layer="1"/>
 <wire x1="20.574" y1="4.826" x2="18.796" y2="3.048" width="0.4064" layer="1"/>
-<wire x1="18.796" y1="3.048" x2="14.478" y2="3.048" width="0.4064" layer="1"/>
+<contactref element="U$2" pad="E"/>
+<wire x1="18.288" y1="5.08" x2="18.288" y2="3.302" width="0.4064" layer="1"/>
+<wire x1="18.288" y1="3.302" x2="18.542" y2="3.048" width="0.4064" layer="1"/>
+<wire x1="9.144" y1="3.048" x2="18.542" y2="3.048" width="0.4064" layer="1"/>
 </signal>
 <signal name="N$18">
@@
 <contactref element="R1" pad="1"/>
 <contactref element="T1" pad="C"/>
-<contactref element="Q1" pad="1"/>
 <wire x1="1.524" y1="13.716" x2="1.524" y2="13.208" width="0.4064" layer="1"/>
-<wire x1="1.524" y1="13.208" x2="1.524" y2="6.858" width="0.4064" layer="1"/>
-<wire x1="1.524" y1="6.858" x2="1.778" y2="6.604" width="0.4064" layer="1"/>
 <wire x1="10.922" y1="10.16" x2="9.906" y2="10.16" width="0.4064" layer="1"/>
 <wire x1="9.906" y1="10.16" x2="9.144" y2="9.398" width="0.4064" layer="1"/>
-<wire x1="9.144" y1="9.398" x2="6.096" y2="9.398" width="0.4064" layer="1"/>
+<wire x1="9.144" y1="9.398" x2="7.366" y2="9.398" width="0.4064" layer="1"/>
+<wire x1="7.366" y1="9.398" x2="6.096" y2="9.398" width="0.4064" layer="1"/>
 <wire x1="6.096" y1="9.398" x2="5.08" y2="10.414" width="0.4064" layer="1"/>
 <wire x1="5.08" y1="10.414" x2="5.08" y2="12.192" width="0.4064" layer="1"/>
 <wire x1="5.08" y1="12.192" x2="4.064" y2="13.208" width="0.4064" layer="1"/>
 <wire x1="4.064" y1="13.208" x2="1.524" y2="13.208" width="0.4064" layer="1"/>
+<wire x1="7.112" y1="9.144" x2="7.366" y2="9.398" width="0.4064" layer="1"/>
+<contactref element="U$3" pad="C"/>
+<wire x1="7.112" y1="6.096" x2="7.112" y2="9.144" width="0.4064" layer="1"/>
 </signal>
 <signal name="N$17">
@@
 <signal name="VIN">
 <contactref element="R1" pad="2"/>
-<contactref element="Q1" pad="3"/>
 <contactref element="T3" pad="C"/>
 <contactref element="JP2" pad="1"/>
 <wire x1="10.922" y1="18.288" x2="10.922" y2="20.066" width="0.4064" layer="1"/>
 <wire x1="10.922" y1="20.066" x2="11.938" y2="21.082" width="0.4064" layer="1"/>
-<wire x1="6.858" y1="6.604" x2="6.858" y2="13.462" width="0.4064" layer="16"/>
-<wire x1="6.858" y1="13.462" x2="6.604" y2="13.716" width="0.4064" layer="16"/>
 <wire x1="6.604" y1="13.716" x2="6.604" y2="13.97" width="0.4064" layer="16"/>
 <wire x1="6.604" y1="13.97" x2="10.922" y2="18.288" width="0.4064" layer="16"/>
+<wire x1="8.382" y1="8.382" x2="6.858" y2="8.382" width="0.4064" layer="16"/>
+<wire x1="6.858" y1="8.382" x2="6.35" y2="8.89" width="0.4064" layer="16"/>
+<wire x1="6.35" y1="8.89" x2="6.35" y2="13.462" width="0.4064" layer="16"/>
+<wire x1="6.35" y1="13.462" x2="6.604" y2="13.716" width="0.4064" layer="16"/>
+<contactref element="U$3" pad="B"/>
+<wire x1="9.652" y1="6.096" x2="9.652" y2="7.112" width="0.4064" layer="16"/>
+<wire x1="9.652" y1="7.112" x2="8.382" y2="8.382" width="0.4064" layer="16"/>
 </signal>
 <signal name="VOUT">
-<contactref element="Q1" pad="2"/>
 <contactref element="R2" pad="2"/>
-<contactref element="U2" pad="3"/>
 <contactref element="C4" pad="1"/>
 <contactref element="R9" pad="2"/>
-<wire x1="3.302" y1="10.922" x2="3.302" y2="7.62" width="0.4064" layer="1"/>
-<wire x1="3.302" y1="7.62" x2="4.318" y2="6.604" width="0.4064" layer="1"/>
-<wire x1="4.318" y1="6.604" x2="4.318" y2="5.334" width="0.4064" layer="1"/>
-<wire x1="4.318" y1="5.334" x2="5.588" y2="4.064" width="0.4064" layer="1"/>
-<wire x1="5.588" y1="4.064" x2="11.43" y2="4.064" width="0.4064" layer="1"/>
-<wire x1="11.43" y1="4.064" x2="12.7" y2="5.334" width="0.4064" layer="1"/>
-<wire x1="23.114" y1="6.096" x2="20.32" y2="6.096" width="0.4064" layer="1"/>
-<wire x1="20.32" y1="6.096" x2="19.05" y2="7.366" width="0.4064" layer="1"/>
-<wire x1="19.05" y1="7.366" x2="13.208" y2="7.366" width="0.4064" layer="1"/>
-<wire x1="13.208" y1="7.366" x2="12.7" y2="6.858" width="0.4064" layer="1"/>
-<wire x1="12.7" y1="6.858" x2="12.7" y2="5.334" width="0.4064" layer="1"/>
 <wire x1="23.114" y1="6.096" x2="32.766" y2="6.096" width="0.4064" layer="1"/>
 <wire x1="32.766" y1="6.096" x2="33.02" y2="6.35" width="0.4064" layer="1"/>
+<wire x1="18.796" y1="6.858" x2="21.59" y2="6.858" width="0.4064" layer="1"/>
+<wire x1="21.59" y1="6.858" x2="22.352" y2="6.096" width="0.4064" layer="1"/>
+<wire x1="22.352" y1="6.096" x2="23.114" y2="6.096" width="0.4064" layer="1"/>
+<wire x1="3.302" y1="10.922" x2="3.302" y2="7.366" width="0.4064" layer="1"/>
+<contactref element="U$2" pad="B"/>
+<wire x1="5.842" y1="4.064" x2="12.192" y2="4.064" width="0.4064" layer="1"/>
+<wire x1="12.192" y1="4.064" x2="13.208" y2="5.08" width="0.4064" layer="1"/>
+<wire x1="13.208" y1="5.08" x2="13.208" y2="6.096" width="0.4064" layer="1"/>
+<wire x1="13.208" y1="6.096" x2="14.478" y2="7.366" width="0.4064" layer="1"/>
+<wire x1="14.478" y1="7.366" x2="18.288" y2="7.366" width="0.4064" layer="1"/>
+<wire x1="18.288" y1="7.366" x2="18.796" y2="6.858" width="0.4064" layer="1"/>
+<contactref element="U$3" pad="E"/>
+<wire x1="4.572" y1="6.096" x2="3.302" y2="7.366" width="0.4064" layer="1"/>
+<wire x1="5.842" y1="4.064" x2="4.572" y2="5.334" width="0.4064" layer="1"/>
+<wire x1="4.572" y1="5.334" x2="4.572" y2="6.096" width="0.4064" layer="1"/>
 </signal>
 <signal name="VON">

Commit message: fixed the names
Parts:
- renumbered U$2 to U2, U$3 to U3
Changed lines of the file:
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@@
 <attribute name="VALUE" x="39.37" y="15.621" size="1.27" layer="27"/>
 </element>
-<element name="U$2" library="dm_parts" package="TO92-BCE" value="L4931" x="15.748" y="5.08"/>
-<element name="U$3" library="dm_parts" package="TO92-BCE" value="VP2206N3-G" x="7.112" y="6.096" rot="R180"/>
+<element name="U2" library="dm_parts" package="TO92-BCE" value="L4931" x="15.748" y="5.08" smashed="yes">
+<attribute name="NAME" x="20.574" y="4.318" size="1.27" layer="25" ratio="10" rot="R90"/>
+<attribute name="VALUE" x="13.208" y="1.778" size="1.27" layer="27" ratio="10"/>
+</element>
+<element name="U3" library="dm_parts" package="TO92-BCE" value="VP2206N3-G" x="7.112" y="6.096" smashed="yes" rot="R180">
+<attribute name="NAME" x="2.286" y="7.62" size="1.27" layer="25" ratio="10" rot="R270"/>
+<attribute name="VALUE" x="9.652" y="9.398" size="1.27" layer="27" ratio="10" rot="R180"/>
+</element>
 </elements>
 <signals>
@@
 <contactref element="C5" pad="-"/>
 <contactref element="R9" pad="1"/>
-<contactref element="U$2" pad="C"/>
+<contactref element="U2" pad="C"/>
 </signal>
 <signal name="AREF">
@@
 <wire x1="24.13" y1="4.826" x2="20.574" y2="4.826" width="0.4064" layer="1"/>
 <wire x1="20.574" y1="4.826" x2="18.796" y2="3.048" width="0.4064" layer="1"/>
-<contactref element="U$2" pad="E"/>
+<contactref element="U2" pad="E"/>
 <wire x1="18.288" y1="5.08" x2="18.288" y2="3.302" width="0.4064" layer="1"/>
 <wire x1="18.288" y1="3.302" x2="18.542" y2="3.048" width="0.4064" layer="1"/>
@@
 <wire x1="4.064" y1="13.208" x2="1.524" y2="13.208" width="0.4064" layer="1"/>
 <wire x1="7.112" y1="9.144" x2="7.366" y2="9.398" width="0.4064" layer="1"/>
-<contactref element="U$3" pad="C"/>
+<contactref element="U3" pad="C"/>
 <wire x1="7.112" y1="6.096" x2="7.112" y2="9.144" width="0.4064" layer="1"/>
 </signal>
@@
 <wire x1="6.35" y1="8.89" x2="6.35" y2="13.462" width="0.4064" layer="16"/>
 <wire x1="6.35" y1="13.462" x2="6.604" y2="13.716" width="0.4064" layer="16"/>
-<contactref element="U$3" pad="B"/>
+<contactref element="U3" pad="B"/>
 <wire x1="9.652" y1="6.096" x2="9.652" y2="7.112" width="0.4064" layer="16"/>
 <wire x1="9.652" y1="7.112" x2="8.382" y2="8.382" width="0.4064" layer="16"/>
@@
 <wire x1="22.352" y1="6.096" x2="23.114" y2="6.096" width="0.4064" layer="1"/>
 <wire x1="3.302" y1="10.922" x2="3.302" y2="7.366" width="0.4064" layer="1"/>
-<contactref element="U$2" pad="B"/>
+<contactref element="U2" pad="B"/>
 <wire x1="5.842" y1="4.064" x2="12.192" y2="4.064" width="0.4064" layer="1"/>
 <wire x1="12.192" y1="4.064" x2="13.208" y2="5.08" width="0.4064" layer="1"/>
@@
 <wire x1="14.478" y1="7.366" x2="18.288" y2="7.366" width="0.4064" layer="1"/>
 <wire x1="18.288" y1="7.366" x2="18.796" y2="6.858" width="0.4064" layer="1"/>
-<contactref element="U$3" pad="E"/>
+<contactref element="U3" pad="E"/>
 <wire x1="4.572" y1="6.096" x2="3.302" y2="7.366" width="0.4064" layer="1"/>
 <wire x1="5.842" y1="4.064" x2="4.572" y2="5.334" width="0.4064" layer="1"/>
