File: power-wing.sch (EAGLE design)
At the start: 25 parts, among them Q1 MOSFET-PGDS_TO220V, T1 2N2222, T2 2N2222, T3 2N2222, U1 TLV2462IP, U2 LD1117

Commit message: off switch to GPIO11 instead of 12 since that is used for sleep
Connections:
- removed net N$19: MS1.GPIO11
- new net GPIO11: MS1.GPIO11, R3.2
- net GPIO12: no longer R3.2
Changed lines of the file:
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@@
 <wire x1="35.56" y1="73.66" x2="35.56" y2="63.5" width="0.1524" layer="91"/>
-</segment>
-<segment>
-<pinref part="R3" gate="G$1" pin="2"/>
-<wire x1="68.58" y1="99.06" x2="63.5" y2="99.06" width="0.1524" layer="91"/>
-<label x="60.96" y="99.06" size="1.778" layer="95"/>
-</segment>
-</net>
-<net name="N$19" class="0">
-<segment>
-<pinref part="MS1" gate="G$1" pin="GPIO11"/>
-<wire x1="38.1" y1="73.66" x2="38.1" y2="63.5" width="0.1524" layer="91"/>
 </segment>
 </net>
@@
 </segment>
 </net>
+<net name="GPIO11" class="0">
+<segment>
+<pinref part="R3" gate="G$1" pin="2"/>
+<wire x1="68.58" y1="99.06" x2="63.5" y2="99.06" width="0.1524" layer="91"/>
+<label x="60.96" y="99.06" size="1.778" layer="95"/>
+</segment>
+<segment>
+<pinref part="MS1" gate="G$1" pin="GPIO11"/>
+<wire x1="38.1" y1="73.66" x2="38.1" y2="63.5" width="0.1524" layer="91"/>
+</segment>
+</net>

Commit message: lets use some smaller parts
Parts:
- removed Q1: MOSFET-PGDS_TO220V, adafruit:MOSFET-PGDS_TO220V
- removed U2: LD1117, dm_parts:LD1117
- added U$2: L4931, dm_parts:L4931
- added U$3: VP2206N3-G, dm_parts:VP2206N3-G
Connections:
- net 3V: now also U$2.VOUT; no longer U2.OUT
- net GND: now also U$2.GND; no longer U2.GND
- net N$16: now also U$3.G; no longer Q1.G
- net VIN: now also U$3.S; no longer Q1.S
- net VOUT: now also U$2.VIN, U$3.D; no longer Q1.D, U2.IN
Other:
- moved on the sheet: C5
Changed lines of the file:
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@@
 <part name="C1" library="adafruit" deviceset="C-US" device="025-024X044" value="2.2u"/>
 <part name="D1" library="diode" deviceset="ZENER-DIODE" device="DO34-7" value="5.2"/>
-<part name="Q1" library="adafruit" deviceset="MOSFET-P" device="GDS_TO220V"/>
 <part name="GND3" library="supply1" deviceset="GND" device=""/>
 <part name="GND4" library="supply1" deviceset="GND" device=""/>
@@
 <part name="R7" library="pot" deviceset="TRIM_EU-" device="PTSPIN" value="1M"/>
 <part name="JP2" library="adafruit" deviceset="PINHD-1X3" device=""/>
-<part name="U2" library="dm_parts" deviceset="LD1117" device=""/>
 <part name="GND7" library="supply1" deviceset="GND" device=""/>
 <part name="C4" library="adafruit" deviceset="C-US" device="025-024X044" value=".1u"/>
@@
 <part name="JP1" library="adafruit" deviceset="PINHD-1X6" device=""/>
 <part name="JP3" library="adafruit" deviceset="PINHD-1X3" device=""/>
+<part name="U$2" library="dm_parts" deviceset="L4931" device=""/>
+<part name="U$3" library="dm_parts" deviceset="VP2206N3-G" device=""/>
 </parts>
 <sheets>
@@
 <instance part="C1" gate="G$1" x="187.96" y="119.38"/>
 <instance part="D1" gate="G$1" x="203.2" y="119.38" rot="R90"/>
-<instance part="Q1" gate="G$1" x="83.82" y="139.7" rot="R90"/>
 <instance part="GND3" gate="1" x="177.8" y="83.82"/>
 <instance part="GND4" gate="1" x="193.04" y="91.44"/>
@@
 <instance part="R7" gate="1" x="187.96" y="96.52"/>
 <instance part="JP2" gate="A" x="58.42" y="152.4"/>
-<instance part="U2" gate="G$1" x="152.4" y="154.94"/>
-<instance part="GND7" gate="1" x="152.4" y="137.16"/>
+<instance part="GND7" gate="1" x="157.48" y="137.16"/>
 <instance part="C4" gate="G$1" x="137.16" y="149.86"/>
-<instance part="C5" gate="G$1" x="167.64" y="149.86"/>
+<instance part="C5" gate="G$1" x="180.34" y="149.86"/>
 <instance part="R9" gate="G$1" x="124.46" y="134.62" rot="R90"/>
 <instance part="GND8" gate="1" x="124.46" y="127"/>
@@
 <instance part="JP1" gate="A" x="45.72" y="7.62" rot="R270"/>
 <instance part="JP3" gate="A" x="50.8" y="76.2" rot="R90"/>
+<instance part="U$2" gate="G$1" x="157.48" y="152.4"/>
+<instance part="U$3" gate="G$1" x="83.82" y="137.16" rot="R90"/>
 </instances>
 <busses>
@@
 </segment>
 <segment>
-<pinref part="U2" gate="G$1" pin="GND"/>
-<wire x1="152.4" y1="142.24" x2="152.4" y2="139.7" width="0.1524" layer="91"/>
+<wire x1="157.48" y1="142.24" x2="157.48" y2="139.7" width="0.1524" layer="91"/>
 <pinref part="GND7" gate="1" pin="GND"/>
 <pinref part="C4" gate="G$1" pin="2"/>
 <wire x1="137.16" y1="144.78" x2="137.16" y2="142.24" width="0.1524" layer="91"/>
-<wire x1="137.16" y1="142.24" x2="152.4" y2="142.24" width="0.1524" layer="91"/>
-<junction x="152.4" y="142.24"/>
-<wire x1="152.4" y1="142.24" x2="167.64" y2="142.24" width="0.1524" layer="91"/>
+<wire x1="137.16" y1="142.24" x2="157.48" y2="142.24" width="0.1524" layer="91"/>
+<junction x="157.48" y="142.24"/>
 <pinref part="C5" gate="G$1" pin="-"/>
-<wire x1="167.64" y1="142.24" x2="167.64" y2="144.78" width="0.1524" layer="91"/>
+<wire x1="157.48" y1="142.24" x2="180.34" y2="142.24" width="0.1524" layer="91"/>
+<wire x1="180.34" y1="142.24" x2="180.34" y2="144.78" width="0.1524" layer="91"/>
+<pinref part="U$2" gate="G$1" pin="GND"/>
+<junction x="157.48" y="142.24"/>
 </segment>
 <segment>
@@
 </segment>
 <segment>
-<pinref part="U2" gate="G$1" pin="OUT"/>
-<wire x1="165.1" y1="154.94" x2="167.64" y2="154.94" width="0.1524" layer="91"/>
 <pinref part="C5" gate="G$1" pin="+"/>
-<wire x1="167.64" y1="154.94" x2="177.8" y2="154.94" width="0.1524" layer="91"/>
-<wire x1="167.64" y1="152.4" x2="167.64" y2="154.94" width="0.1524" layer="91"/>
-<junction x="167.64" y="154.94"/>
+<wire x1="180.34" y1="154.94" x2="190.5" y2="154.94" width="0.1524" layer="91"/>
+<wire x1="180.34" y1="152.4" x2="180.34" y2="154.94" width="0.1524" layer="91"/>
+<pinref part="U$2" gate="G$1" pin="VOUT"/>
+<wire x1="172.72" y1="154.94" x2="180.34" y2="154.94" width="0.1524" layer="91"/>
+<junction x="180.34" y="154.94"/>
 </segment>
 </net>
@@
 <pinref part="T1" gate="G$1" pin="C"/>
 <wire x1="81.28" y1="129.54" x2="81.28" y2="127" width="0.1524" layer="91"/>
-<pinref part="Q1" gate="G$1" pin="G"/>
-<wire x1="81.28" y1="134.62" x2="81.28" y2="129.54" width="0.1524" layer="91"/>
+<pinref part="U$3" gate="G$1" pin="G"/>
 <junction x="81.28" y="129.54"/>
 </segment>
@@
 <pinref part="R1" gate="G$1" pin="2"/>
 <wire x1="66.04" y1="139.7" x2="55.88" y2="139.7" width="0.1524" layer="91"/>
-<pinref part="Q1" gate="G$1" pin="S"/>
-<wire x1="66.04" y1="139.7" x2="78.74" y2="139.7" width="0.1524" layer="91"/>
+<label x="55.88" y="139.7" size="1.778" layer="95"/>
+<wire x1="76.2" y1="139.7" x2="66.04" y2="139.7" width="0.1524" layer="91"/>
 <junction x="66.04" y="139.7"/>
-<label x="55.88" y="139.7" size="1.778" layer="95"/>
+<pinref part="U$3" gate="G$1" pin="S"/>
 </segment>
 <segment>
@@
 <net name="VOUT" class="0">
 <segment>
-<pinref part="Q1" gate="G$1" pin="D"/>
 <pinref part="R2" gate="G$1" pin="2"/>
-<wire x1="88.9" y1="139.7" x2="101.6" y2="139.7" width="0.1524" layer="91"/>
 <wire x1="101.6" y1="139.7" x2="124.46" y2="139.7" width="0.1524" layer="91"/>
-<junction x="101.6" y="139.7"/>
 <wire x1="124.46" y1="139.7" x2="124.46" y2="154.94" width="0.1524" layer="91"/>
-<pinref part="U2" gate="G$1" pin="IN"/>
 <wire x1="124.46" y1="154.94" x2="137.16" y2="154.94" width="0.1524" layer="91"/>
 <pinref part="C4" gate="G$1" pin="1"/>
-<wire x1="137.16" y1="154.94" x2="139.7" y2="154.94" width="0.1524" layer="91"/>
 <wire x1="137.16" y1="152.4" x2="137.16" y2="154.94" width="0.1524" layer="91"/>
-<junction x="137.16" y="154.94"/>
 <pinref part="R9" gate="G$1" pin="2"/>
 <junction x="124.46" y="139.7"/>
-</segment>
-</net>
+<wire x1="93.98" y1="139.7" x2="101.6" y2="139.7" width="0.1524" layer="91"/>
+<junction x="101.6" y="139.7"/>
+<pinref part="U$2" gate="G$1" pin="VIN"/>
+<wire x1="139.7" y1="154.94" x2="137.16" y2="154.94" width="0.1524" layer="91"/>
+<junction x="137.16" y="154.94"/>
+<pinref part="U$3" gate="G$1" pin="D"/>
+</segment>
+</net>

Commit message: fixed the names
Parts:
- renumbered U$2 to U2, U$3 to U3
Changed lines of the file:
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@@
 <part name="JP1" library="adafruit" deviceset="PINHD-1X6" device=""/>
 <part name="JP3" library="adafruit" deviceset="PINHD-1X3" device=""/>
-<part name="U$2" library="dm_parts" deviceset="L4931" device=""/>
-<part name="U$3" library="dm_parts" deviceset="VP2206N3-G" device=""/>
+<part name="U2" library="dm_parts" deviceset="L4931" device=""/>
+<part name="U3" library="dm_parts" deviceset="VP2206N3-G" device=""/>
 </parts>
 <sheets>
@@
 <instance part="JP1" gate="A" x="45.72" y="7.62" rot="R270"/>
 <instance part="JP3" gate="A" x="50.8" y="76.2" rot="R90"/>
-<instance part="U$2" gate="G$1" x="157.48" y="152.4"/>
-<instance part="U$3" gate="G$1" x="83.82" y="137.16" rot="R90"/>
+<instance part="U2" gate="G$1" x="157.48" y="152.4"/>
+<instance part="U3" gate="G$1" x="83.82" y="137.16" rot="R90"/>
 </instances>
 <busses>
@@
 <wire x1="157.48" y1="142.24" x2="180.34" y2="142.24" width="0.1524" layer="91"/>
 <wire x1="180.34" y1="142.24" x2="180.34" y2="144.78" width="0.1524" layer="91"/>
-<pinref part="U$2" gate="G$1" pin="GND"/>
+<pinref part="U2" gate="G$1" pin="GND"/>
 <junction x="157.48" y="142.24"/>
 </segment>
@@
 <wire x1="180.34" y1="154.94" x2="190.5" y2="154.94" width="0.1524" layer="91"/>
 <wire x1="180.34" y1="152.4" x2="180.34" y2="154.94" width="0.1524" layer="91"/>
-<pinref part="U$2" gate="G$1" pin="VOUT"/>
+<pinref part="U2" gate="G$1" pin="VOUT"/>
 <wire x1="172.72" y1="154.94" x2="180.34" y2="154.94" width="0.1524" layer="91"/>
 <junction x="180.34" y="154.94"/>
@@
 <pinref part="T1" gate="G$1" pin="C"/>
 <wire x1="81.28" y1="129.54" x2="81.28" y2="127" width="0.1524" layer="91"/>
-<pinref part="U$3" gate="G$1" pin="G"/>
+<pinref part="U3" gate="G$1" pin="G"/>
 <junction x="81.28" y="129.54"/>
 </segment>
@@
 <wire x1="76.2" y1="139.7" x2="66.04" y2="139.7" width="0.1524" layer="91"/>
 <junction x="66.04" y="139.7"/>
-<pinref part="U$3" gate="G$1" pin="S"/>
+<pinref part="U3" gate="G$1" pin="S"/>
 </segment>
 <segment>
@@
 <wire x1="93.98" y1="139.7" x2="101.6" y2="139.7" width="0.1524" layer="91"/>
 <junction x="101.6" y="139.7"/>
-<pinref part="U$2" gate="G$1" pin="VIN"/>
+<pinref part="U2" gate="G$1" pin="VIN"/>
 <wire x1="139.7" y1="154.94" x2="137.16" y2="154.94" width="0.1524" layer="91"/>
 <junction x="137.16" y="154.94"/>
-<pinref part="U$3" gate="G$1" pin="D"/>
-</segment>
-</net>
+<pinref part="U3" gate="G$1" pin="D"/>
+</segment>
+</net>
